File: hw/control_board/control_board.kicad_sch (KiCad schematic)
At the start: 49 parts, among them Q1 AOD4189, Q2 BSS138, Q3 SS8050, Q4 SS8050, SW1 B3U-3000PM-B, U1 ESP32-WROOM-32E, U2 DRV8251A, U3 AP63203WU, U4 74LVC2G17

Commit message: control_board schema update
Parts:
- C10: value 1u -> 100n
Changed lines of the file:
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@@
 			)
 		)
-		(property "Value" "1u"
+		(property "Value" "100n"
 			(at 349.758 51.054 0)
 			(show_name no)
