File: hw_v2.0/control_board/control_board.kicad_pcb (KiCad board)
At the start: 2 copper layers, 64 x 69.9 mm, 58 parts, among them J6 Micro_SD_Card, Q1 AOD4189, Q2 BSS138, Q3 SS8050, Q4 SS8050, SW1 B3U-3000PM-B, SW2 SKRPABE010, SW3 SKRPABE010, U1 ESP32-WROOM-32E, U2 DRV8251A, U3 AP63203WU, U4 74LVC2G17

Commit message: limit sw filter added
Parts:
- added C11: 10n, Capacitor_SMD:C_0805_2012Metric, F.Cu at (82.3, 71.4)
- added C13: 10n, Capacitor_SMD:C_0805_2012Metric, F.Cu at (82.3, 75.1)
- added C14: 100n, Capacitor_SMD:C_0805_2012Metric_Pad1.18x1.45mm_HandSolder, B.Cu at (109.9, 76.3)
- added JP1: SolderJumper_3_Open, Jumper:SolderJumper-3_P1.3mm_Open_RoundedPad1.0x1.5mm_NumberLabels, B.Cu at (101.6, 62.2)
- added R22: 1k, Resistor_SMD:R_0805_2012Metric, F.Cu at (80.0, 71.4)
- added R23: 1k, Resistor_SMD:R_0805_2012Metric, F.Cu at (80.0, 75.1)
- C9: value 100n -> 1u
- moved R9 9.41 mm to (73.4, 78.2), turned to 0 degrees
- moved R8 5.97 mm to (77.1, 78.2), turned to 0 degrees
- moved J3 2.79 mm to (76.5, 68.6)
- moved J1 1.38 mm to (76.4, 84.2)
Connections:
- U1 pad 14: /SD_MISO -> /SD_MISO_B
- U1 pad 27: unconnected-(U1-IO16-Pad27) -> /SD_MISO_A
- U4 pad 1: /LSW_1 -> Net-(C11-Pad1)
- U4 pad 3: /LSW_2 -> Net-(C13-Pad1)
Routing:
- net /SD_MISO_A: track 0.00 -> 15.2 mm, vias 0 -> 1
- net +3.3V: track 231.5 -> 243.2 mm
- net Net-(C13-Pad1): track 0.00 -> 7.93 mm
- net Net-(C11-Pad1): track 0.00 -> 6.43 mm
- net /LSW_2: track 12.9 -> 7.37 mm
- net /SD_MISO_B: track 0.00 -> 5.37 mm, vias 0 -> 1
- net /LSW_1: track 14.7 -> 10.9 mm
- net /SD_MISO: track 25.5 -> 28.1 mm, vias 0 -> 1
- net Net-(J1-Pin_2): track 9.91 -> 8.31 mm
- net GND: track 50.6 -> 51.8 mm, vias 33 -> 35
- net VM: track 25.8 -> 24.8 mm
- net Net-(J1-Pin_1): track 14.3 -> 13.5 mm
Other:
- board text added: "IO12"
- board text added: "IO16"
