File: hw_v2.0/control_board/control_board.kicad_sch (KiCad schematic)
At the start: 58 parts, among them J6 Micro_SD_Card, Q1 AOD4189, Q2 BSS138, Q3 SS8050, Q4 SS8050, SW1 B3U-3000PM-B, SW2 SKRPABE010, SW3 SKRPABE010, U1 ESP32-WROOM-32E, U2 DRV8251A, U3 AP63203WU, U4 74LVC2G17

Commit message: limit sw filter added
Parts:
- added C11, C13: 10n, Capacitor_SMD:C_0805_2012Metric, symbol Device:C
- added C14: 100n, Capacitor_SMD:C_0805_2012Metric_Pad1.18x1.45mm_HandSolder, symbol Device:C
- added JP1: SolderJumper_3_Open, Jumper:SolderJumper-3_P1.3mm_Open_RoundedPad1.0x1.5mm_NumberLabels, symbol Jumper:SolderJumper_3_Open
- added R22, R23: 1k, Resistor_SMD:R_0805_2012Metric, symbol Device:R
- C9: value 100n -> 1u
- R1, R19, R20: now not fitted
Connections:
- net +3.3V: now also C14.1
- net GND: now also C11.2, C13.2, C14.2
- net LSW_1: now also R22.2; no longer U4.1
- net LSW_2: now also R23.2; no longer U4.3
- net SD_MISO: now also JP1.2 (C); no longer U1.14 (IO12)
- net SD_MISO_A: now reaches U1.27 (IO16)
- net SD_MISO_A: now also JP1.3 (B)
- new net: C11.1, R22.1, U4.1
- new net: C13.1, R23.1, U4.3
- new net SD_MISO_B: JP1.1 (A), U1.14 (IO12)
- no-connect marks 9 -> 8
Other:
- moved on the sheet: U4A, U4B
