File: hw_v2.0/control_board/control_board.kicad_sch (KiCad schematic)
At the start: 64 parts, among them J6 Micro_SD_Card, Q1 AOD4189, Q2 BSS138, Q3 SS8050, Q4 SS8050, SW1 B3U-3000PM-B, SW2 SKRPABE010, SW3 SKRPABE010, U1 ESP32-WROOM-32E, U2 DRV8251A, U3 AP63203WU, U4 74LVC2G17

Commit message: added sensor connector labels
Parts:
- J6: value Micro_SD_Card -> GCT_MEM2067-02-180-00-A_REVB
- U1: value ESP32-WROOM-32E -> ESP32-WROOM-32E-N4
Changed lines of the file:
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@@
 			)
 		)
-		(property "Value" "Micro_SD_Card"
+		(property "Value" "GCT_MEM2067-02-180-00-A_REVB"
 			(at 361.315 179.07 0)
 			(show_name no)
@@
 			)
 		)
-		(property "Value" "ESP32-WROOM-32E"
+		(property "Value" "ESP32-WROOM-32E-N4"
 			(at 367.9033 81.28 0)
 			(show_name no)
