File: hw_v2.0/snimac/snimac.kicad_pcb (KiCad board)
At the start: 2 copper layers, 78 x 20 mm, 11 parts, among them J1 Conn_01x04, Q1 EE-SX1106, Q2 EE-SX1106

Commit message: limit sw filter added
Parts:
- moved Q2 4.00 mm to (155.0, 56.0)
- moved R2 4.00 mm to (147.5, 60.0)
- moved R3 4.00 mm to (147.5, 57.0)
Routing:
- net /LSW_1: track 15.3 -> 19.3 mm
Other:
- board text added: "LIMIT SWITCH PCB VER 2.0"
- board text removed: "LIMIT SWITCH PCB VER 1.0"
Changed lines of the file:
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@@
 		(capping no)
 		(filling no)
-		(zone_defaults)
 		(aux_axis_origin 97.75 58.5)
 		(grid_origin 97.75 58.5)
@@
 	(footprint "_my_switches:EESX1106"
 		(layer "F.Cu")
-		(at 159 56 -90)
+		(at 155 56 -90)
 		(descr "EE-SX1106")
 		(tags "Phototransistor")
@@
 		)
 		(property "Value" "Conn_01x04"
-			(at 3 4 90)
+			(at 3 8 90)
 			(layer "F.Fab")
 			(effects
@@
 	(footprint "Resistor_SMD:R_0805_2012Metric_Pad1.20x1.40mm_HandSolder"
 		(layer "F.Cu")
-		(at 151.5 57)
+		(at 147.5 57)
 		(descr "Resistor SMD 0805 (2012 Metric), square (rectangular) end terminal, IPC-7351 nominal with elongated pad for handsoldering. (Body size source: IPC-SM-782 page 72, https://www.pcb-3d.com/wordpress/wp-content/uploads/ipc-sm-782a_amendment_1_and_2.pdf)")
 		(tags "resistor handsolder")
@@
 	(footprint "Resistor_SMD:R_0805_2012Metric_Pad1.20x1.40mm_HandSolder"
 		(layer "F.Cu")
-		(at 151.5 60)
+		(at 147.5 60)
 		(descr "Resistor SMD 0805 (2012 Metric), square (rectangular) end terminal, IPC-7351 nominal with elongated pad for handsoldering. (Body size source: IPC-SM-782 page 72, https://www.pcb-3d.com/wordpress/wp-content/uploads/ipc-sm-782a_amendment_1_and_2.pdf)")
 		(tags "resistor handsolder")
@@
 		(layer "Edge.Cuts")
 	)
-	(gr_text "LIMIT SWITCH PCB VER 1.0"
+	(gr_text "LIMIT SWITCH PCB VER 2.0"
 		(at 111.75 68 0)
 		(layer "F.SilkS")
@@
 	)
 	(segment
-		(start 150.5 57)
-		(end 105 57)
+		(start 147.788 55.579)
+		(end 146.5 56.867)
 		(width 0.5)
 		(layer "F.Cu")
@@
 	)
 	(segment
-		(start 161.5 55.5)
-		(end 159.75 53.75)
+		(start 149.566 55.579)
+		(end 147.788 55.579)
 		(width 0.5)
 		(layer "F.Cu")
@@
 	)
 	(segment
-		(start 159.75 53.75)
-		(end 153.75 53.75)
+		(start 155.75 53.75)
+		(end 151.395 53.75)
 		(width 0.5)
 		(layer "F.Cu")
@@
 	)
 	(segment
+		(start 146.5 57)
+		(end 105 57)
+		(width 0.5)
+		(layer "F.Cu")
+		(net "+3.3V")
+	)
+	(segment
+		(start 151.395 53.75)
+		(end 149.566 55.579)
+		(width 0.5)
+		(layer "F.Cu")
+		(net "+3.3V")
+	)
+	(segment
+		(start 146.5 56.867)
+		(end 146.5 57)
+		(width 0.5)
+		(layer "F.Cu")
+		(net "+3.3V")
+	)
+	(segment
+		(start 146.5 57)
+		(end 146.5 60)
+		(width 0.5)
+		(layer "F.Cu")
+		(net "+3.3V")
+	)
+	(segment
+		(start 157.5 55.5)
+		(end 155.75 53.75)
+		(width 0.5)
+		(layer "F.Cu")
+		(net "+3.3V")
+	)
+	(segment
 		(start 164.95 55.5)
-		(end 161.5 55.5)
+		(end 157.5 55.5)
 		(width 0.5)
 		(layer "F.Cu")
@@
 	)
 	(segment
-		(start 150.5 57)
-		(end 150.5 60)
-		(width 0.5)
-		(layer "F.Cu")
-		(net "+3.3V")
-	)
-	(segment
-		(start 153.75 53.75)
-		(end 150.5 57)
-		(width 0.5)
-		(layer "F.Cu")
-		(net "+3.3V")
-	)
-	(segment
-		(start 159 61.375)
-		(end 159 61)
+		(start 103 60.75)
+		(end 103 60)
+		(width 0.5)
+		(layer "F.Cu")
+		(net "/LSW_2")
+	)
+	(segment
+		(start 157.25 61.5)
+		(end 155.5 63.25)
+		(width 0.5)
+		(layer "F.Cu")
+		(net "/LSW_2")
+	)
+	(segment
+		(start 164.95 61.5)
+		(end 157.25 61.5)
+		(width 0.5)
+		(layer "F.Cu")
+		(net "/LSW_2")
+	)
+	(segment
+		(start 97.5 63)
+		(end 100.75 63)
+		(width 0.5)
+		(layer "F.Cu")
+		(net "/LSW_2")
+	)
+	(segment
+		(start 151.395 63.25)
+		(end 149.645 61.5)
+		(width 0.5)
+		(layer "F.Cu")
+		(net "/LSW_2")
+	)
+	(segment
+		(start 96.5 61)
+		(end 96.5 62)
+		(width 0.5)
+		(layer "F.Cu")
+		(net "/LSW_2")
+	)
+	(segment
+		(start 96.5 62)
+		(end 97.5 63)
+		(width 0.5)
+		(layer "F.Cu")
+		(net "/LSW_2")
+	)
+	(segment
+		(start 100.75 63)
+		(end 103 60.75)
+		(width 0.5)
+		(layer "F.Cu")
+		(net "/LSW_2")
+	)
+	(segment
+		(start 149.645 61.5)
+		(end 102.25 61.5)
+		(width 0.5)
+		(layer "F.Cu")
+		(net "/LSW_2")
+	)
+	(segment
+		(start 155.5 63.25)
+		(end 151.395 63.25)
+		(width 0.5)
+		(layer "F.Cu")
+		(net "/LSW_2")
+	)
+	(segment
+		(start 155 56)
+		(end 155.5 56)
+		(width 0.5)
+		(layer "F.Cu")
+		(net "/LSW_1")
+	)
+	(segment
+		(start 159 59.5)
+		(end 164.95 59.5)
+		(width 0.5)
+		(layer "F.Cu")
+		(net "/LSW_1")
+	)
+	(segment
+		(start 149.669 57)
+		(end 151.919 54.75)
+		(width 0.5)
+		(layer "F.Cu")
+		(net "/LSW_1")
+	)
+	(segment
+		(start 151.919 54.75)
+		(end 153.75 54.75)
+		(width 0.5)
+		(layer "F.Cu")
+		(net "/LSW_1")
+	)
+	(segment
+		(start 148.5 57)
+		(end 149.669 57)
+		(width 0.5)
+		(layer "F.Cu")
+		(net "/LSW_1")
+	)
+	(segment
+		(start 155.5 56)
+		(end 159 59.5)
+		(width 0.5)
+		(layer "F.Cu")
+		(net "/LSW_1")
+	)
+	(segment
+		(start 153.75 54.75)
+		(end 155 56)
+		(width 0.5)
+		(layer "F.Cu")
+		(net "/LSW_1")
+	)
+	(segment
+		(start 148.5 60)
+		(end 149.542 60)
 		(width 0.5)
 		(layer "F.Cu")
@@
 	)
 	(segment
-		(start 152.5 60)
-		(end 154.75 62.25)
+		(start 155 61.375)
+		(end 155 61)
 		(width 0.5)
 		(layer "F.Cu")
@@
 	)
 	(segment
-		(start 158.125 62.25)
-		(end 159 61.375)
+		(start 154.125 62.25)
+		(end 155 61.375)
 		(width 0.5)
 		(layer "F.Cu")
@@
 	)
 	(segment
-		(start 154.75 62.25)
-		(end 158.125 62.25)
+		(start 149.542 60)
+		(end 151.792 62.25)
+		(width 0.5)
+		(layer "F.Cu")
+		(net "Net-(Q2-A)")
+	)
+	(segment
+		(start 151.792 62.25)
+		(end 154.125 62.25)
 		(width 0.5)
 		(layer "F.Cu")
@@
 		(net "Net-(Q1-A)")
 	)
-	(segment
-		(start 159 56)
-		(end 159.5 56)
-		(width 0.5)
-		(layer "F.Cu")
-		(net "/LSW_1")
-	)
-	(segment
-		(start 154.75 54.75)
-		(end 157.75 54.75)
-		(width 0.5)
-		(layer "F.Cu")
-		(net "/LSW_1")
-	)
-	(segment
-		(start 157.75 54.75)
-		(end 159 56)
-		(width 0.5)
-		(layer "F.Cu")
-		(net "/LSW_1")
-	)
-	(segment
-		(start 163 59.5)
-		(end 164.95 59.5)
-		(width 0.5)
-		(layer "F.Cu")
-		(net "/LSW_1")
-	)
-	(segment
-		(start 159.5 56)
-		(end 163 59.5)
-		(width 0.5)
-		(layer "F.Cu")
-		(net "/LSW_1")
-	)
-	(segment
-		(start 152.5 57)
-		(end 154.75 54.75)
-		(width 0.5)
-		(layer "F.Cu")
-		(net "/LSW_1")
-	)
-	(segment
-		(start 154.25 63.25)
-		(end 152.5 61.5)
-		(width 0.5)
-		(layer "F.Cu")
-		(net "/LSW_2")
-	)
-	(segment
-		(start 103 60.75)
-		(end 103 60)
-		(width 0.5)
-		(layer "F.Cu")
-		(net "/LSW_2")
-	)
-	(segment
-		(start 161.25 61.5)
-		(end 159.5 63.25)
-		(width 0.5)
-		(layer "F.Cu")
-		(net "/LSW_2")
-	)
-	(segment
-		(start 97.5 63)
-		(end 100.75 63)
-		(width 0.5)
-		(layer "F.Cu")
-		(net "/LSW_2")
-	)
-	(segment
-		(start 96.5 61)
-		(end 96.5 62)
-		(width 0.5)
-		(layer "F.Cu")
-		(net "/LSW_2")
-	)
-	(segment
-		(start 159.5 63.25)
-		(end 154.25 63.25)
-		(width 0.5)
-		(layer "F.Cu")
-		(net "/LSW_2")
-	)
-	(segment
-		(start 96.5 62)
-		(end 97.5 63)
-		(width 0.5)
-		(layer "F.Cu")
-		(net "/LSW_2")
-	)
-	(segment
-		(start 164.95 61.5)
-		(end 161.25 61.5)
-		(width 0.5)
-		(layer "F.Cu")
-		(net "/LSW_2")
-	)
-	(segment
-		(start 100.75 63)
-		(end 103 60.75)
-		(width 0.5)
-		(layer "F.Cu")
-		(net "/LSW_2")
-	)
-	(segment
-		(start 152.5 61.5)
-		(end 102.25 61.5)
-		(width 0.5)
-		(layer "F.Cu")
-		(net "/LSW_2")
-	)
 	(zone

Commit message: added sensor connector labels
Parts:
- moved J1 3.45 mm to (161.5, 55.6)
Routing:
- net /LSW_2: track 73.7 -> 70.3 mm
- net /LSW_1: track 19.3 -> 15.9 mm
- net +3.3V: track 68.1 -> 64.7 mm
Other:
- board text added: "3V3"
- board text added: "GND"
- board text added: "LS1"
- board text added: "LS2"
